File: Nodes/TempHumNode/Hardware/temphum_node/temphum_node.kicad_sch (KiCad schematic)
At the start: 62 parts, among them IC1 CC1310F128RGZR, IC2 TPD6E004RSER, J1 TC2050-IDC, U1 MCP73123-22SI/MF, U2 SHT35-DIS-B, U3 TPS22860DBVR, U4 TPS63900DSKR, U5 MCP3421A0T-E/CH, Y2 TSX-3225 24.0000MF15X-AC3, Y3 FC-135_32.7680KA-AG0

Commit message: hw(temphum-node): wire MCP3421 battery-SoC ADC + gated divider
MCP3421 (0x68) on 3V3_SW, VIN-=GND, VIN+=1M/1M 0.1% divider tap (Ctap
10nF). Divider high-side gated by a 2nd TPS22860 (BAT+->BAT+_SW, ON=
PERIPH_EN, VBIAS=VIN=BAT+): ~18nA guaranteed leakage, tap collapses to
~0 in sleep so VIN+ can't back-leak into the off ADC. Chosen over a
complementary MOSFET pair (uncertain 1uA IDSS max).

Co-Authored-By: Claude Opus 4.8 (1M context) <noreply@anthropic.com>
Parts:
- added C27, C28: 100nF, symbol Device:C
- added C29: 10nF, symbol Device:C
- added R11, R12: 1M 0.1%, symbol Device:R
- added U6: TPS22860DBVR, SmartHome:SOT-23-6_L2.9-W1.6-P0.95-LS2.8-BR, symbol SmartHome:TPS22860DBVR
Connections:
- net VCC is gone; now on net 3V3: U3.4 (VIN), U3.5 (VBIAS)
- net 3V3: now also C27.1
- net BAT+: now also C28.1, U6.4 (VIN), U6.5 (VBIAS)
- net GND: now also U5.2 (VSS), U5.6 (Vin-), C27.2, C28.2, C29.2, R12.1, U6.2 (GND)
- net SCL: now also U5.3 (SCL)
- net SDA: now also U5.4 (SDA)
- net VCC_SWITCH: no longer C22.1, R3.2, R4.2, R5.2, U2.2 (ADDR), U2.5 (VDD), U3.1 (VOUT)
- net at U5.1 (Vin+): now also C29.1, R11.2, R12.2
- net 3V3_SW: now reaches U5.5 (VDD)
- net 3V3_SW: now also C22.1, R3.2, R4.2, R5.2, U2.2 (ADDR), U2.5 (VDD), U3.1 (VOUT)
- net DRV_OUT renamed PERIPH_EN
- net PERIPH_EN: now also U6.6 (ON)
- new net BAT+_SW: R11.1, U6.1 (VOUT)
- no-connect marks 36 -> 37
Other:
- moved on the sheet: U5

Commit message: hw(temphum-node): CC1310 support parts - pogo/ESD 3D, crystal swaps
Add TC2030-IDC UART pogo (SnapEDA, both footprints + 3D, symbol made
SmartHome-native). Attach TPD6E004 ESD 3D model + merge its symbol into
SmartHome. Add in-stock crystal replacements: ECS-240-9-33B (24MHz 9pF,
capless HF) and Epson FC-135R (32.768kHz 12.5pF, 2x12pF caps) - both CL/
ESR-matched drop-ins. Plus CC1310 schematic GPIO/pogo wiring.

Co-Authored-By: Claude Opus 4.8 (1M context) <noreply@anthropic.com>
Parts:
- removed Y2: TSX-3225 24.0000MF15X-AC3, SmartHome:TSX3225240000MF15XAC3, symbol SmartSwitch:TSX-3225_24.0000MF20G-AC3
- removed Y3: FC-135_32.7680KA-AG0, SmartHome:FC135327680KAAG0, symbol FC-135_32_7680KA-AG0:FC-135_32.7680KA-AG0
- added TC1: TC2030-IDC, SmartHome:TC2030-IDC, symbol SmartHome:TC2030-IDC
- added U7: ECS-240-9-33B-CWN-TR, SmartHome:CRYSTAL-SMD_4P-L3.2-W2.5-BL, symbol SmartHome:ECS-240-9-33B-CWN-TR
- added X1: FC-135R, SmartHome:OSC-SMD_L3.2-W1.5, symbol SmartHome:FC-135R
- C1: value C -> 2.2nF
Connections:
- net VCC_SWITCH is gone; now on net 3V3: R1.1
- net GND: now also TC1.1, U7.2 (Gnd), U7.4 (Gnd)
- net PERIPH_EN: now also IC1.10 (DIO_5)
- net SCL: now also IC1.6 (DIO_1)
- net SDA: now also IC1.7 (DIO_2)
- net nBUTTON: now also IC1.11 (DIO_6)
- net nCHRGSTAT: now also IC1.12 (DIO_7)
- net at C9.1, IC1.4 (X32K_Q1): now also X1.1 (OSC1)
- net at C14.1, IC1.5 (X32K_Q2): now also X1.2 (OSC2)
- net at IC1.47 (X24M_P): now also U7.1 (In/Out)
- net at IC1.46 (X24M_N): now also U7.3 (Out/In)
- net UART_TX: now reaches IC1.8 (DIO_3)
- net UART_TX: now also TC1.2
- net UART_RX: now reaches IC1.9 (DIO_4)
- net UART_RX: now also TC1.3
- net LED_BLUE: no longer names the net of IC1.38 (DIO_25)
- net LED_RED: no longer names the net of IC1.37 (DIO_24)
- net RELAY1: no longer names the net of IC1.40 (DIO_27)
- net TOUCH_OUT: no longer names the net of IC1.39 (DIO_26)
Other:
- moved on the sheet: AE1, C14, C16, C17, C18, C19, C20, C21, C4, C5, C6, C7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

Commit message: hw(temphum-node): passive footprints/3D, ferrite/inductor/LED/0805 parts
Add ferrite bead BLM18HE152 (L0603), DCDC inductor MLZ2012N6R8 (IND-
SMD), 0805 cap footprint, red LED XL-1608SURC (LED0603). Attach 3D
models to the perfected passive footprints (C_0402, C_0603, R_0603,
L_Polarized_0402) - library + all placed board instances; R_0603 model
orientation fixed (rotate 0 0 -90). Node schematic essentially
complete; only the battery connector remains before layout.

Co-Authored-By: Claude Opus 4.8 (1M context) <noreply@anthropic.com>
Parts:
- removed L8: BLM18HE152SN1D, SmartHome:BLM18SP221SN1B, symbol SmartSwitch:L
- removed L9: 6.8uH, SmartHome:MLZ2012N6R8LT000_0805, symbol SmartSwitch:L
- added L11: MLZ2012N6R8LT000, SmartHome:IND-SMD_L2.0-W1.3, symbol SmartHome:MLZ2012N6R8LT000
- added L8: BLM18HE152SN1D, SmartHome:L0603, symbol SmartHome:BLM18HE152SN1D
- C1, C2, C23, C24: footprint (none) -> SmartHome:C_0603
- C17, C19: LCSC C105226 -> C86295
- C22: footprint CC0603KRX7R9BB104:CAPC1608X90N -> SmartHome:C_0603; LCSC C14663 -> C1591
- C26: footprint (none) -> SmartHome:C_0603; LCSC (none) -> C86295
- C27, C28, C29, C3: footprint (none) -> SmartHome:C_0402
- D2: footprint (none) -> SmartHome:LED0603-RD_RED; LCSC (none) -> C965799
- R1, R10, R11, R12, R2, R6, R7, R8, R9: footprint (none) -> SmartHome:R_0603
- R3, R4, R5: footprint CRCW060310K0FKEA:RESC1608X50N -> SmartHome:R_0603; LCSC (none) -> C844918
Connections:
- net 3V3: now also L8.1
- net DCDC_SW: now also L11.1
- net VDDR: now also L11.2
- net VDDS: now also L8.2
