File: Nodes/TempHumNode/Hardware/temphum_node/temphum_node.kicad_sch (KiCad schematic)
At the start: 69 parts, among them IC1 CC1310F128RGZR, IC2 TPD6E004RSER, J1 TC2050-IDC, U1 MCP73123-22SI/MF, U2 SHT35-DIS-B, U3 TPS22860DBVR, U4 TPS63900DSKR, U5 MCP3421A0T-E/CH, U6 TPS22860DBVR, U7 ECS-240-9-33B-CWN-TR, X1 FC-135R

Commit message: hw(temphum-node): add battery connector (JST B2B-PH-K-S placeholder)
Add JST PH 2.0mm 2-pin top-entry THT connector (LCSC C131337) as the
battery input placeholder. Top-entry chosen (lead internal to the
enclosure). To be confirmed against the actual pack Tue: connector
family (PH vs XH) + which pin is BAT+.

Co-Authored-By: Claude Opus 4.8 (1M context) <noreply@anthropic.com>
Parts:
- added CN1: B2B-PH-K-S, SmartHome:CONN-TH_B2B-PH-K-S, symbol SmartHome:B2B-PH-K-S
Connections:
- net BAT+: now also CN1.1
- net GND: now also CN1.2
Other:
- note added: "3V3 REGULATOR"
- note added: "BATTERY SOCKET"
- note added: "BATTERY VOLTAGE MEASUREMENT CIRCUIT"
- note added: "JOIN BUTTON"
- note added: "LiFePO4 CHARGER"
- note added: "MCU (CC1310) with Antenna"
- note added: "MCU UART Interface POGO pad"
- note added: "PERIPHERIAL POWER SWITCH"
- note added: "SHT35 I2C TEMPERATURE SENSOR"
- note added: "USB-C with ESD PROTECTION (PWR Only)"
- moved on the sheet: AE1, C1, C10, C11, C12, C13, C14, C15, C16, C17, C18, C19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

Commit message: hw(temphum): rev2 node schematic + PCB layout + KiCad lib parts
Full rev-2 T&H node hardware: wired schematic, 4-layer PCB layout
(RF-first placement, GND stitching, DRC-clean). Library additions:
JST XH 2.5mm connector (C158012), R_0402, and imported/perfected
footprints. USB-C center holes fixed to NPTH (annular-ring clean).

Co-Authored-By: Claude Opus 4.8 (1M context) <noreply@anthropic.com>
Parts:
- removed CN1: B2B-PH-K-S, SmartHome:CONN-TH_B2B-PH-K-S, symbol SmartHome:B2B-PH-K-S
- added CN2: B2B-XH-A, SmartHome:CONN-TH_B2B-XH-A-LF-SN, symbol SmartHome:B2B-XH-A
- C25: footprint SmartHome:C_0603 -> SmartHome:C_0402
- R13: footprint SmartHome:R_0603 -> SmartHome:R_0402
Connections:
- net BAT+: now also CN2.1
- net CC1: now also D1.3, D1.4; no longer D1.1, D1.6
- net CC2: now also D1.1, D1.6; no longer D1.3, D1.4
- net GND: now also CN2.2
- net JTAG_TDI: now also IC1.27 (DIO_17); no longer IC1.26 (DIO_16)
- net JTAG_TDO: now also IC1.26 (DIO_16); no longer IC1.21 (DIO_15)
- net PERIPH_EN: now also IC1.38 (DIO_25); no longer IC1.10 (DIO_5)
- net SCL: now also IC1.15 (DIO_9); no longer IC1.6 (DIO_1)
- net SDA: now also IC1.16 (DIO_10); no longer IC1.7 (DIO_2)
- net UART_RX: now also IC1.19 (DIO_13); no longer IC1.9 (DIO_4)
- net UART_TX: now also IC1.18 (DIO_12), TC1.5; no longer IC1.8 (DIO_3), TC1.2
- net nBUTTON: now also IC1.39 (DIO_26); no longer IC1.11 (DIO_6)
- net nCHRGSTAT: now also IC1.20 (DIO_14); no longer IC1.12 (DIO_7)

Commit message: hw(temphum): rev2 production-ready — sent to JLCPCB
Footprints refined to TI/Microchip datasheets: CC1310 EP paste windowpane
(dodges thermal vias) + 0.24mm roundrect pads + NSMD 0.05; DFN charger &
WSON regulator EP paste segmentation; USB-C center holes NPTH + 0.65 drill.
XH battery connector, AITRONIC logo, GND stitching, silkscreen. Full LCSC
BOM + CPL + Gerbers (3 assembled protos ordered).

Co-Authored-By: Claude Opus 4.8 (1M context) <noreply@anthropic.com>
Parts:
- C1: LCSC Part (none) -> C86023
- C10: LCSC C76963 -> (none); LCSC Part (none) -> C76963
- C11, C12: LCSC C913745 -> (none); LCSC Part (none) -> C913745
- C13, C6: LCSC C77177 -> (none); LCSC Part (none) -> C77177
- C14, C9: LCSC C76948 -> (none); LCSC Part (none) -> C76948
- C15: LCSC C29266 -> (none); LCSC Part (none) -> C29266
- C16, C18, C20, C21, C4, C5: LCSC C60474 -> (none); LCSC Part (none) -> C60474
- C17, C19, C26: LCSC C86295 -> (none); LCSC Part (none) -> C86295
- C2, C23: LCSC Part (none) -> C86016
- C22: LCSC C1591 -> (none); LCSC Part (none) -> C1591
- C24: LCSC Part (none) -> C91606
- C25: LCSC C106861 -> (none); LCSC Part (none) -> C106861
- C27, C28, C3: LCSC Part (none) -> C60474
- C29: LCSC Part (none) -> C77019
- C7: LCSC C88891 -> (none); LCSC Part (none) -> C88891
- C8: LCSC C41744 -> (none); LCSC Part (none) -> C41744
- D2: LCSC C965799 -> (none); LCSC Part (none) -> C965799
- IC1: LCSC C84353 -> (none); LCSC Part (none) -> C84353
- IC2: LCSC C1973052 -> (none); LCSC Part (none) -> C1973052
- L1: LCSC C98003 -> (none); LCSC Part (none) -> C98003
- L2, L3, L4: LCSC C77110 -> (none); LCSC Part (none) -> C77110
- L5, L7: LCSC C98001 -> (none); LCSC Part (none) -> C98001
- L6: LCSC C12669 -> (none); LCSC Part (none) -> C12669
- R1: LCSC Part (none) -> C23061
- R10: LCSC Part (none) -> C23029
- R11, R12: LCSC Part (none) -> C4250208
- R13: LCSC C25896 -> (none); LCSC Part (none) -> C25896
- R2, R6: LCSC Part (none) -> C2907044
- R3, R4, R5: LCSC C844918 -> (none); LCSC Part (none) -> C844918
- R7: LCSC Part (none) -> C2907033
- R8: LCSC Part (none) -> C2906980
- R9: LCSC Part (none) -> C2907002
